Commit message: ros

File: SPEAR_Arm.urdf (robot description, URDF)
Before this commit: robot SPEAR_Arm, 8 links, 7 joints
Joints:
- joint Elbow Roll: axis 1 0 0 -> (none); limit lower=-3.1416 upper=3.1416 effort=0 velocity=0 -> (none); origin xyz=0 0.09 0 rpy=0 0 0 -> xyz=0 0.0782 0 rpy=0 0 0; type revolute -> fixed
