Commit message: Description of Arm Complete

File: description/URDF/SPEAR_Arm.urdf (robot description, URDF)
Before this commit: robot kipps_arm, 0 links, 0 joints
Links:
- added link base_drum; visual mesh filename=package://description/meshes/base_drum.stl
- added link base_link; visual mesh filename=package://description/meshes/base_link.stl
- added link link1; visual mesh filename=package://description/meshes/link1.stl
- added link link2; visual mesh filename=package://description/meshes/link2.stl
- added link link3; visual mesh filename=package://description/meshes/link3.stl
- added link link4; visual mesh filename=package://description/meshes/link4.stl
- added link link5; visual mesh filename=package://description/meshes/link5.stl
Joints:
- added joint base_joint: type revolute, parent base_link, child base_drum, origin xyz=0 0 0.03935 rpy=0 0 0, axis 0 0 1, limit lower=0.00 upper=3.14159 effort=1000.0 velocity=50.0
- added joint eef_joint: type fixed, parent link4, child link5, origin xyz=0.099 0.06567 0.0 rpy=0.0 0.0 0.0
- added joint link1_joint: type revolute, parent base_drum, child link1, origin xyz=0 0.0019 0.07018 rpy=0 0 0, axis 0 1 0, limit lower=-3.14159 upper=3.14159 effort=1000.0 velocity=50.0
- added joint link2_joint: type revolute, parent link1, child link2, origin xyz=0.34315 0.01784 0 rpy=0 0 0, axis 0 1 0, limit lower=-3.14159 upper=3.14159 effort=1000.0 velocity=50.0
- added joint link3_joint: type revolute, parent link2, child link3, origin xyz=0.01450 -0.08525 0 rpy=0 0 0, axis 1 0 0, limit lower=-3.14159 upper=3.14159 effort=1000.0 velocity=50.0
- added joint link4_joint: type revolute, parent link3, child link4, origin xyz=0.24068 0.013 0 rpy=0 0 0, axis 0 1 0, limit lower=-3.14159 upper=3.14159 effort=1000.0 velocity=50.0
