Commit message: Zed Camera Added, File Restructred

File: src/kipp_description/src/description/kipp.urdf (robot description, URDF)
Before this commit: robot kipp, 11 links, 10 joints
Joints:
- added joint $(arg camera_name_2)_joint: type fixed, parent base_link, child $(arg camera_name_2)_camera_link, origin xyz=-0.4 0.0 0.25 rpy=0 0 ${M_PI}
- joint back_left_wheel_joint: axis 0 0 0 -> 0 0 1
- joint back_right_wheel_joint: axis 0 0 0 -> 0 0 1
- joint front_left_wheel_joint: axis 0 0 0 -> 0 0 1
- joint front_right_wheel_joint: axis 0 0 0 -> 0 0 1
- joint middle_left_wheel_joint: axis 0 0 0 -> 0 0 1; origin xyz=0 0.25 -0.25 rpy=0 0 0 -> xyz=0 -0.25 -0.25 rpy=0 0 0
- joint middle_right_wheel_joint_: axis 0 0 0 -> 0 0 1; origin xyz=0 -0.25 -0.25 rpy=0 0 0 -> xyz=0 0.25 -0.25 rpy=0 0 0
