Commit message: GPS working with Zed

File: src/kipp_description/src/kipp.urdf (robot description, URDF)
Before this commit: robot kipp, 11 links, 11 joints
Links:
- added link gnss_link; visual cylinder length=0.05 radius=0.05
Joints:
- added joint gnss_joint: type fixed, parent base_link, child gnss_link, origin xyz=0 0 0.70 rpy=0 0 0
